File: Instrument Equalizer/Rockman EQ.kicad_pcb (KiCad board)
At the start: 2 copper layers, 216 x 127 mm, 123 parts, among them IC101 TL072, IC102 TL072, IC103 TL072, IC104 TL072, IC105 TL072, IC106 TL072, IC107 TL072, IC108 TL072, IC201 TL072, IC301 LM339

Commit message: Passive Components placed
Parts:
- added D506: 1N4148, Rockman:Resistor-Capacitor, F.Cu at (235.2, 140.8)
- added Q301: MMBFJ112, Package_TO_SOT_THT:TO-92_Wide, F.Cu at (172.1, 94.6)
- added Q501: L7912, Package_TO_SOT_THT:TO-220-3_Vertical, F.Cu at (74.2, 148.4)
- added Q502: L7812, Package_TO_SOT_THT:TO-220-3_Vertical, F.Cu at (92.7, 148.1)
- added Q503: MMBFJ112, Package_TO_SOT_THT:TO-92_Wide, F.Cu at (240.7, 138.2)
- moved R314 367.4 mm to (234.7, 108.3)
- moved R313 358.3 mm to (222.7, 104.5)
- moved R106 351.2 mm to (244.5, 61.8)
- moved R102 350.0 mm to (228.6, 61.7)
- moved R103 349.0 mm to (231.3, 61.7)
- moved R104 348.1 mm to (234.0, 61.7)
- moved R105 347.2 mm to (236.8, 61.8)
- moved C304 335.2 mm to (231.6, 108.3)
- moved R226 326.0 mm to (227.8, 85.7)
- moved R227 325.3 mm to (230.7, 85.6)
- moved C213 324.5 mm to (210.9, 71.4)
- moved R511 324.4 mm to (245.7, 140.9)
- moved R407 322.3 mm to (207.4, 122.8)
- moved R408 321.5 mm to (210.2, 122.7)
- moved C212 320.1 mm to (202.8, 71.4)
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