File: Octopus/Octopus.kicad_sch (KiCad schematic)
At the start: 54 parts, among them J1 MIDI IN (to panel DIN), J10 RN111PC, J2 9-12VDC IN, J3 RN111PC, J4 RN111PC, J5 RN111PC, J6 RN111PC, J7 RN111PC, J8 RN111PC, J9 RN111PC, K1 G5V-1, K2 G5V-1, K3 G5V-1, K4 G5V-1, K5 G5V-1, K6 G5V-1, K7 G5V-1, K8 G5V-1, U1 Teensy4.1, U2 6N138, U3 ULN2803A, U4 L7805

Commit message: Octopus updates
Parts:
- removed H3, H4: M3, MountingHole:MountingHole_3.2mm_M3, symbol Mechanical:MountingHole
- added C1: 10uF 25V, Capacitor_THT:CP_Radial_D6.3mm_P2.50mm, symbol Device:C_Polarized
- added C2: 22uF 10V, Capacitor_THT:CP_Radial_D6.3mm_P2.50mm, symbol Device:C_Polarized
- added J11: Button panel, Connector_JST:JST_XH_B6B-XH-A_1x06_P2.50mm_Vertical, symbol Connector_Generic:Conn_01x06
- added JP10, JP11, JP12, JP13, JP14, JP15, JP16, JP9: NO|NC, Jumper:SolderJumper-3_P1.3mm_Bridged12_RoundedPad1.0x1.5mm, symbol Jumper:SolderJumper_3_Bridged12
- added K10, K11, K12, K13, K14, K15, K16, K9: G5V-1, Relay_THT:Relay_SPDT_Omron_G5V-1, symbol Relay:G5V-1
- added LED10, LED11, LED12, LED13, LED14, LED15, LED16, LED9: LED, LED_THT:LED_D3.0mm, symbol Device:LED
- added R109, R110, R111, R112, R113, R114, R115, R116: 1k, Resistor_THT:R_Axial_DIN0207_L6.3mm_D2.5mm_P2.54mm_Vertical, symbol Device:R
- added U5: ULN2803A, Package_DIP:DIP-18_W7.62mm, symbol Transistor_Array:ULN2803A
- J10, J3, J4, J5, J6, J7, J8, J9: value RN111PC -> RN112BPC; footprint Octopus:Jack_6.35mm_Switchcraft_RN111PC_Vertical -> Octopus:Jack_6.35mm_Switchcraft_RN112BPC_Horizontal; symbol Connector_Audio:AudioJack2 -> Connector_Audio:AudioJack3
- J2: footprint Connector_BarrelJack:BarrelJack_Horizontal -> TerminalBlock_Phoenix:TerminalBlock_Phoenix_MKDS-1,5-2-5.08_1x02_P5.08mm_Horizontal; symbol Connector:Barrel_Jack -> Connector:Screw_Terminal_01x02
- R101, R102, R103, R104, R105, R106, R107, R108: footprint Resistor_THT:R_Axial_DIN0207_L6.3mm_D2.5mm_P10.16mm_Horizontal -> Resistor_THT:R_Axial_DIN0207_L6.3mm_D2.5mm_P2.54mm_Vertical
- U4: value L7805 -> R-78E5.0-1.0; footprint Package_TO_SOT_THT:TO-220-3_Vertical -> Converter_DCDC:Converter_DCDC_RECOM_R-78E-0.5_THT; symbol Regulator_Linear:L7805 -> Converter_DCDC:R-78E5.0-0.5
Connections:
- net +3V3: now also J11.2 (Pin_2)
- net +5V: now also C2.1, J11.1 (Pin_1), K10.2, K11.2, K12.2, K13.2, K14.2, K15.2, K16.2, K9.2, R109.1, R110.1, R111.1, R112.1, R113.1, R114.1, R115.1, R116.1, U5.10 (COM)
- net GND: now also C1.2, C2.2, J11.3 (Pin_3), U5.9 (GND)
- net DRV3: now reaches K3.9, LED3.1 (K), U3.13 (O6)
- net at F1.2, U4.1 (IN): now also C1.1
- net DRV6: now reaches K6.9, LED6.1 (K), U3.16 (O3)
- net DRV7: now reaches K7.9, LED7.1 (K), U3.17 (O2)
- net DRV8: now reaches K8.9, LED8.1 (K), U3.18 (O1)
- net DRV5: now reaches K5.9, LED5.1 (K), U3.15 (O4)
- net DRV1: now reaches K1.9, LED1.1 (K), U3.11 (O8)
- net DRV2: now reaches K2.9, LED2.1 (K), U3.12 (O7)
- net DRV4: now reaches K4.9, LED4.1 (K), U3.14 (O5)
- net CH1_COM renamed JACK1_SLV
- net JACK1_SLV: now also K9.5, K9.6
- net CH1_TIP renamed CH1_OUT
- net CH2_COM renamed JACK2_SLV
- net JACK2_SLV: now also K10.5, K10.6
- net CH2_TIP renamed CH2_OUT
- net CH3_COM renamed JACK3_SLV
- net JACK3_SLV: now also K11.5, K11.6
- net CH3_TIP renamed CH3_OUT
- net CH4_COM renamed JACK4_SLV
- net JACK4_SLV: now also K12.5, K12.6
- net CH4_TIP renamed CH4_OUT
- net CH5_COM renamed JACK5_SLV
- net JACK5_SLV: now also K13.5, K13.6
- net CH5_TIP renamed CH5_OUT
- net CH6_COM renamed JACK6_SLV
- net JACK6_SLV: now also K14.5, K14.6
- net CH6_TIP renamed CH6_OUT
- net CH7_COM renamed JACK7_SLV
- net JACK7_SLV: now also K15.5, K15.6
- net CH7_TIP renamed CH7_OUT
- net CH8_COM renamed JACK8_SLV
- net JACK8_SLV: now also K16.5, K16.6
- net CH8_TIP renamed CH8_OUT
- new net: LED14.2 (A), R114.2
- new net: LED15.2 (A), R115.2
- new net: LED11.2 (A), R111.2
- new net: LED9.2 (A), R109.2
- new net: U1.31 (IO31), U5.1 (I1)
- new net: U1.30 (IO30), U5.2 (I2)
- new net: U1.29 (IO29), U5.3 (I3)
- new net: U1.28 (IO28), U5.4 (I4)
- new net: U1.27 (IO27), U5.5 (I5)
- new net: U1.26 (IO26), U5.6 (I6)
- new net: U1.25 (IO25), U5.7 (I7)
- new net: U1.24 (IO24), U5.8 (I8)
- new net: LED13.2 (A), R113.2
- new net: LED10.2 (A), R110.2
- new net: LED12.2 (A), R112.2
- new net: LED16.2 (A), R116.2
- new net CH10_NC: JP10.3 (B), K10.1
- new net CH10_NO: JP10.1 (A), K10.10
- new net CH10_OUT: J4.R, JP10.2 (C)
- new net CH11_NC: JP11.3 (B), K11.1
- new net CH11_NO: JP11.1 (A), K11.10
- new net CH11_OUT: J5.R, JP11.2 (C)
- new net CH12_NC: JP12.3 (B), K12.1
- new net CH12_NO: JP12.1 (A), K12.10
- new net CH12_OUT: J6.R, JP12.2 (C)
- new net CH13_NC: JP13.3 (B), K13.1
- new net CH13_NO: JP13.1 (A), K13.10
- new net CH13_OUT: J7.R, JP13.2 (C)
- new net CH14_NC: JP14.3 (B), K14.1
- new net CH14_NO: JP14.1 (A), K14.10
- new net CH14_OUT: J8.R, JP14.2 (C)
- new net CH15_NC: JP15.3 (B), K15.1
- new net CH15_NO: JP15.1 (A), K15.10
- new net CH15_OUT: J9.R, JP15.2 (C)
- new net CH16_NC: JP16.3 (B), K16.1
- new net CH16_NO: JP16.1 (A), K16.10
- new net CH16_OUT: J10.R, JP16.2 (C)
- new net CH9_NC: JP9.3 (B), K9.1
- new net CH9_NO: JP9.1 (A), K9.10
- new net CH9_OUT: J3.R, JP9.2 (C)
- new net DRV10: K10.9, LED10.1 (K), U5.12 (O7)
- new net DRV11: K11.9, LED11.1 (K), U5.13 (O6)
- new net DRV12: K12.9, LED12.1 (K), U5.14 (O5)
- new net DRV13: K13.9, LED13.1 (K), U5.15 (O4)
- new net DRV14: K14.9, LED14.1 (K), U5.16 (O3)
- new net DRV15: K15.9, LED15.1 (K), U5.17 (O2)
- new net DRV16: K16.9, LED16.1 (K), U5.18 (O1)
- new net DRV9: K9.9, LED9.1 (K), U5.11 (O8)
- new net I2C_SCL: J11.5 (Pin_5), U1.19 (SCL0)
- new net I2C_SDA: J11.4 (Pin_4), U1.18 (SDA0)
- new net PANEL_INT: J11.6 (Pin_6), U1.22 (IO22)
Other:
- moved on the sheet: J2, JP1, JP2, JP3, JP4, JP5, JP6, JP7, JP8, K1, K2, K3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
