File: Octopus/Octopus.kicad_sch (KiCad schematic)
At the start: 61 parts, among them J1 FM6725 MIDI IN, J10 RN112BPC, J11 Button panel, J12 FM6725 MIDI THRU, J2 9-12VDC IN, J3 RN112BPC, J4 RN112BPC, J5 RN112BPC, J6 RN112BPC, J7 RN112BPC, J8 RN112BPC, J9 RN112BPC, K1 G5V-1, K10 G5V-1, K11 G5V-1, K12 G5V-1, K13 G5V-1, K14 G5V-1, K15 G5V-1, K16 G5V-1, K2 G5V-1, K3 G5V-1, K4 G5V-1, K5 G5V-1, K6 G5V-1, K7 G5V-1, K8 G5V-1, K9 G5V-1, U1 Teensy4.1, U2 6N138, U3 ULN2803A, U4 R-78E5.0-1.0, U5 ULN2803A, U6 74HCT14

Commit message: Added standard power supply
Parts:
- removed C1: 10uF 25V, Capacitor_THT:CP_Radial_D6.3mm_P2.50mm, symbol Device:C_Polarized
- removed C2: 22uF 16V, Capacitor_THT:CP_Radial_D6.3mm_P2.50mm, symbol Device:C_Polarized
- removed C3: 100n, Capacitor_THT:C_Disc_D5.0mm_W2.5mm_P5.00mm, symbol Device:C
- removed F1: MF-RHT070 0.7A, Fuse:Fuse_Bourns_MF-RHT070, symbol Device:Polyfuse_Small
- removed J2: 9-12VDC IN, TerminalBlock_Phoenix:TerminalBlock_Phoenix_MKDS-1,5-2-5.08_1x02_P5.08mm_Horizontal, symbol Connector:Screw_Terminal_01x02
- removed U4: R-78E5.0-1.0, Converter_DCDC:Converter_DCDC_RECOM_R-78E-0.5_THT, symbol Converter_DCDC:R-78E5.0-0.5
- added C501: 1000u, Capacitor_THT:CP_Radial_D10.0mm_P5.00mm, symbol Device:C_Polarized
- added C502: 100n, Capacitor_THT:C_Disc_D10.0mm_W2.5mm_P5.00mm, symbol Device:C
- added D2: DF005M, Diode_THT:Diode_Bridge_DIP-4_W7.62mm_P5.08mm, symbol Diode_Bridge:DF005M
- added D505: 1N4001, Diode_THT:D_A-405_P12.70mm_Horizontal, symbol Device:D_Filled
- added F2: Fuse, Fuse:Fuseholder_Littelfuse_100_series_5x30mm, symbol Device:Fuse
- added Q501: L7805, Package_TO_SOT_THT:TO-220-3_Vertical, symbol Regulator_Linear:L7812
- added SW101: NE1838EE, Rockman:NE18_2U_EE_P_6AMP, symbol Switch:SW_Push_DPDT
- added X1: PSS-332, Rockman:Transformer_Hammond_164D_1.1VA, symbol Transformer:TRANSF3
Connections:
- net +5V: now also C502.1, D505.1 (K), Q501.3 (OUT)
- net GND: now also C501.2, C502.2, D2.2 (-), D505.2 (A), Q501.2 (GND), X1.4, X1.5
- new net: F2.1, SW101.3 (C)
- new net: F2.2, X1.1
- new net: C501.1, D2.1 (+), Q501.1 (IN)
- new net: SW101.6 (C), X1.2
- new net: D2.4, X1.3
- new net: D2.3, X1.6
- new net LINE: SW101.2 (B), SW101.5 (B)
Other:
- note added: "Power Supply"
- moved on the sheet: D1, H1, H2, J1, R1, R2, U2, U6A, U6B, U6C
