File: Octopus/panel/OctopusPanel.kicad_sch (KiCad schematic)
At the start: 43 parts, among them J1 To main board J11, SW1 228CMVARGBFDNR, SW2 228CMVARGBFDNR, SW3 228CMVARGBFDNR, SW4 228CMVARGBFDNR, SW5 228CMVARGBFDNR, SW6 228CMVARGBFDNR, SW7 228CMVARGBFDNR, SW8 228CMVARGBFDNR, U1 PCA9685PW, U2 PCA9685PW, U3 MCP23008-xSO

Commit message: Octopus: front-panel display + encoder, Omron B3W-9 buttons, DigiKey BOM
- Button board: 0.96" SSD1306 OLED (Winstar WEA012864D-03 on 5 mm
  spacers) and an Alps EC11E15204A3 encoder with push switch, left of
  the buttons. MCP23008 -> MCP23017 for the extra inputs (GPA7/GPB7
  unused: output-only on current silicon).
- Buttons: the discontinued CTS 228C RGB switches are replaced by Omron
  B3W-9000-RG2N (red + green LEDs): red = tip, green = ring, amber =
  both. One PCA9685 instead of two; LED resistors are four Bourns CAT16
  4-resistor arrays. Square 10.6 mm panel cut-outs.
- Firmware: Display (U8g2/U8x8, redraws only what changed), encoder
  decoding from the MCP23017 interrupt (half-cycle detents), SELECT? /
  push-to-load / 5 s timeout, presets shown and entered as 1-128,
  MidiHandler::recall(), bigger Serial1 RX buffer.
- Main board: status LEDs and their resistors removed (the buttons show
  every line); C2 value corrected to 22 uF 16 V.
- BOM_DigiKey.csv: full parts list by manufacturer part number
  (force-added: the repo ignores *.csv).
- ERC 0 errors on both boards; DRC 0 errors, 0 unconnected, 0 parity
  (main board: 16 vendor-footprint silkscreen-at-edge warnings).

Co-Authored-By: Claude Opus 5.5 <noreply@anthropic.com>
Parts:
- removed R10, R11, R13, R14, R16, R17, R19, R20, R22, R23, R7, R8: 390, Resistor_SMD:R_0805_2012Metric, symbol Device:R
- removed R12, R15, R18, R21, R24, R6, R9: 220, Resistor_SMD:R_0805_2012Metric, symbol Device:R
- removed R25, R26: 4.7k, Resistor_SMD:R_0805_2012Metric, symbol Device:R
- removed U2: PCA9685PW, Package_SO:TSSOP-28_4.4x9.7mm_P0.65mm, symbol Driver_LED:PCA9685PW
- added C6, C7: 10n, Capacitor_SMD:C_0805_2012Metric, symbol Device:C
- added J2: WEA012864D-03 OLED, OctopusPanel:OLED_Winstar_WEA012864D-03, symbol Connector_Generic:Conn_01x04
- added RN1, RN2: 330, Resistor_SMD:R_Array_Convex_4x0603, symbol Device:R_Pack04
- added RN3, RN4: 180, Resistor_SMD:R_Array_Convex_4x0603, symbol Device:R_Pack04
- added SW9: EC11E15204A3, Rotary_Encoder:RotaryEncoder_Alps_EC11E-Switch_Vertical_H20mm, symbol Device:RotaryEncoder_Switch
- C3: value 100n -> 10u
- C5: value 10u -> 10n
- R1, R2: value 390 -> 4.7k
- R3: value 220 -> 10k
- R4, R5: value 390 -> 10k
- SW1, SW2, SW3, SW4, SW5, SW6, SW7, SW8: value 228CMVARGBFDNR -> B3W-9000-RG2N; footprint OctopusPanel:CTS_228CMV_RGB -> OctopusPanel:Omron_B3W-9_2LED_10x10; symbol OctopusPanel:CTS_228C_RGB -> OctopusPanel:B3W-9_RG
- U3: value MCP23008-xSO -> MCP23017; footprint Package_SO:SOIC-18W_7.5x11.6mm_P1.27mm -> Package_SO:SOIC-28W_7.5x17.9mm_P1.27mm; symbol Interface_Expansion:MCP23008-xSO -> Interface_Expansion:MCP23017x-x-SO
Connections:
- net +3V3: now also R1.1, R2.1, R3.1, R4.1, R5.1, U3.9 (V_{DD}), J2.1 (Pin_1); no longer C4.1, U3.6 (~{RESET})
- net +5V: now also C4.1, SW1.A1 (R+), SW1.A2 (G+), SW2.A1 (R+), SW2.A2 (G+), SW3.A1 (R+), SW3.A2 (G+), SW4.A1 (R+), SW4.A2 (G+), SW5.A1 (R+), SW5.A2 (G+), SW6.A1 (R+), SW6.A2 (G+), SW7.A1 (R+), SW7.A2 (G+), SW8.A1 (R+), SW8.A2 (G+); no longer C5.1, SW1.L3 (LED+), SW2.L3 (LED+), SW3.L3 (LED+), SW4.L3 (LED+), SW5.L3 (LED+), SW6.L3 (LED+), SW7.L3 (LED+), SW8.L3 (LED+)
- net BTN1: now also U3.21 (GPA0); no longer U3.10 (GP0)
- net BTN2: now also U3.22 (GPA1); no longer U3.11 (GP1)
- net BTN3: now also U3.23 (GPA2); no longer U3.12 (GP2)
- net BTN4: now also U3.24 (GPA3); no longer U3.13 (GP3)
- net BTN5: now also U3.25 (GPA4); no longer U3.14 (GP4)
- net BTN6: now also U3.26 (GPA5); no longer U3.15 (GP5)
- net BTN7: now also U3.27 (GPA6); no longer U3.16 (GP6)
- net BTN8: now also U3.1 (GPB0); no longer U3.17 (GP7)
- net DRV1_G: now also RN3.8 (R1.2); no longer R2.2
- net DRV1_R: now also RN1.8 (R1.2); no longer R1.2
- net DRV2_G: now also RN3.7 (R2.2); no longer R5.2
- net DRV2_R: now also RN1.7 (R2.2); no longer R4.2
- net DRV3_G: now also RN3.6 (R3.2)
- net DRV3_R: now also RN1.6 (R3.2)
- net DRV4_G: now also RN3.5 (R4.2)
- net DRV4_R: now also RN1.5 (R4.2)
- net DRV5_G: now also RN4.8 (R1.2)
- net DRV5_R: now also RN2.8 (R1.2)
- net DRV6_G: now also RN4.7 (R2.2)
- net DRV6_R: now also RN2.7 (R2.2)
- net DRV7_G: now also RN4.6 (R3.2)
- net DRV7_R: now also RN2.6 (R3.2)
- net DRV8_G: now also RN4.5 (R4.2)
- net DRV8_R: now also RN2.5 (R4.2)
- net GND: now also U3.10 (V_{SS}), U3.15 (A0), U3.16 (A1), U3.17 (A2), C6.2, C7.2, J2.2 (Pin_2), SW9.C, SW9.S2; no longer U3.3 (A2), U3.4 (A1), U3.5 (A0), U3.9 (VSS)
- net LED1_G: now also SW1.K2 (G-), RN3.1 (R1.1); no longer R2.1, SW1.L4 (G)
- net LED1_R: now also SW1.K1 (R-), RN1.1 (R1.1); no longer R1.1, SW1.L2 (R)
- net LED2_G: now also SW2.K2 (G-), RN3.2 (R2.1); no longer R5.1, SW2.L4 (G)
- net LED2_R: now also SW2.K1 (R-), RN1.2 (R2.1); no longer R4.1, SW2.L2 (R)
- net LED3_G: now also SW3.K2 (G-), RN3.3 (R3.1); no longer SW3.L4 (G)
- net LED3_R: now also SW3.K1 (R-), RN1.3 (R3.1); no longer SW3.L2 (R)
- net LED4_G: now also SW4.K2 (G-), RN3.4 (R4.1); no longer SW4.L4 (G)
- net LED4_R: now also SW4.K1 (R-), RN1.4 (R4.1); no longer SW4.L2 (R)
- net LED5_G: now also SW5.K2 (G-), RN4.1 (R1.1); no longer SW5.L4 (G)
- net LED5_R: now also SW5.K1 (R-), RN2.1 (R1.1); no longer SW5.L2 (R)
- net LED6_G: now also SW6.K2 (G-), RN4.2 (R2.1); no longer SW6.L4 (G)
- net LED6_R: now also SW6.K1 (R-), RN2.2 (R2.1); no longer SW6.L2 (R)
- net LED7_G: now also SW7.K2 (G-), RN4.3 (R3.1); no longer SW7.L4 (G)
- net LED7_R: now also SW7.K1 (R-), RN2.3 (R3.1); no longer SW7.L2 (R)
- net LED8_G: now also SW8.K2 (G-), RN4.4 (R4.1); no longer SW8.L4 (G)
- net LED8_R: now also SW8.K1 (R-), RN2.4 (R4.1); no longer SW8.L2 (R)
- net PANEL_INT: now also U3.20 (INTA); no longer U3.8 (INT)
- net SCL: now also R2.2, U3.12 (SCK), J2.3 (Pin_3); no longer U3.1 (SCL)
- net SDA: now also R1.2, U3.13 (SDA), J2.4 (Pin_4); no longer U3.2 (SDA)
- net DRV1_B renamed ENC_A
- net ENC_A: now also C5.1, U3.2 (GPB1), SW9.A
- removed net LED1_B: R3.1, SW1.L1 (B)
- removed net LED2_B: SW2.L1 (B)
- removed net LED3_B: SW3.L1 (B)
- removed net LED4_B: SW4.L1 (B)
- removed net LED5_B: SW5.L1 (B)
- removed net LED6_B: SW6.L1 (B)
- removed net LED7_B: SW7.L1 (B)
- removed net LED8_B: SW8.L1 (B)
- new net ENC_B: C6.1, R4.2, SW9.B, U3.3 (GPB2)
- new net ENC_SW: C7.1, R5.2, SW9.S1, U3.4 (GPB3)
- no-connect marks 9 -> 8
Other:
- moved on the sheet: C5, R1, R2, R3, R4, R5
